File: RP2040_base_example.kicad_pcb (KiCad board)
At the start: 2 copper layers, 21.1 x 45.7 mm, 34 parts, among them J1 Conn_01x03, J2 Conn_01x13, J3 GT-USB-7047C, SW1 SW_Push, U1 XC6206P332MR, U2 SRV05-4, U3 RP2040, U4 W25QXXXJV, Y1 X322512MSB4SI

Commit message: Improve ground path around voltage regulator
Parts:
- turned C1 to 90 degrees
Routing:
- net GND: vias 30 -> 33
Changed lines of the file:
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@@
   )
   (footprint "Capacitor_SMD:C_0603_1608Metric" (layer "F.Cu")
-    (at 68.353827 44 -90)
+    (at 68.353827 44 90)
     (descr "Capacitor SMD 0603 (1608 Metric), square (rectangular) end terminal, IPC_7351 nominal, (Body size source: IPC-SM-782 page 76, https://www.pcb-3d.com/wordpress/wp-content/uploads/ipc-sm-782a_amendment_1_and_2.pdf), generated with kicad-footprint-generator")
     (tags "capacitor")
@@
     (fp_line (start 0.8 0.4) (end -0.8 0.4)
       (stroke (width 0.1) (type solid)) (layer "F.Fab"))
-    (pad "1" smd roundrect (at -0.775 0 270) (size 0.9 0.95) (layers "F.Cu" "F.Paste" "F.Mask") (roundrect_rratio 0.25)
+    (pad "1" smd roundrect (at -0.775 0 90) (size 0.9 0.95) (layers "F.Cu" "F.Paste" "F.Mask") (roundrect_rratio 0.25)
       (net 44 "VBUS") (pintype "passive"))
-    (pad "2" smd roundrect (at 0.775 0 270) (size 0.9 0.95) (layers "F.Cu" "F.Paste" "F.Mask") (roundrect_rratio 0.25)
+    (pad "2" smd roundrect (at 0.775 0 90) (size 0.9 0.95) (layers "F.Cu" "F.Paste" "F.Mask") (roundrect_rratio 0.25)
       (net 3 "GND") (pintype "passive"))
     (model "${KICAD6_3DMODEL_DIR}/Capacitor_SMD.3dshapes/C_0603_1608Metric.wrl"
@@
   (via (at 70.585786 70.585786) (size 0.5) (drill 0.3) (layers "F.Cu" "B.Cu") (free) (net 3))
   (via (at 67.757359 78.363961) (size 0.5) (drill 0.3) (layers "F.Cu" "B.Cu") (free) (net 3))
+  (via (at 63.5 43.815) (size 0.5) (drill 0.3) (layers "F.Cu" "B.Cu") (free) (net 3))
   (via (at 66.696699 82.960155) (size 0.5) (drill 0.3) (layers "F.Cu" "B.Cu") (free) (net 3))
   (via (at 67.403806 67.757359) (size 0.5) (drill 0.3) (layers "F.Cu" "B.Cu") (free) (net 3))
   (via (at 68.110913 62.100505) (size 0.5) (drill 0.3) (layers "F.Cu" "B.Cu") (free) (net 3))
+  (via (at 69.342 43.18) (size 0.5) (drill 0.3) (layers "F.Cu" "B.Cu") (free) (net 3))
   (via (at 76.596194 65.989592) (size 0.5) (drill 0.3) (layers "F.Cu" "B.Cu") (free) (net 3))
   (via (at 80.838835 70.232233) (size 0.5) (drill 0.3) (layers "F.Cu" "B.Cu") (free) (net 3))
@@
   (via (at 70.585786 73.414214) (size 0.5) (drill 0.3) (layers "F.Cu" "B.Cu") (free) (net 3))
   (via (at 76.242641 64.928932) (size 0.5) (drill 0.3) (layers "F.Cu" "B.Cu") (free) (net 3))
+  (via (at 64.77 43.815) (size 0.5) (drill 0.3) (layers "F.Cu" "B.Cu") (free) (net 3))
   (segment (start 78.17538 54.676085) (end 77.467417 54.676085) (width 0.127) (layer "F.Cu") (net 4))
   (segment (start 74.75 51.25) (end 74.75 49.5) (width 0.127) (layer "F.Cu") (net 4))
@@
   (segment (start 66.938037 44.511618) (end 67.01321 44.58679) (width 0.254) (layer "F.Cu") (net 44))
   (segment (start 74.113079 47.9) (end 73.213079 47) (width 0.254) (layer "F.Cu") (net 44))
-  (segment (start 67.067209 44.532791) (end 67.01321 44.58679) (width 0.254) (layer "F.Cu") (net 44))
+  (segment (start 68.111618 44.532791) (end 68.353827 44.775) (width 0.254) (layer "F.Cu") (net 44))
   (segment (start 67.01321 45.16321) (end 68.85 47) (width 0.254) (layer "F.Cu") (net 44))
   (segment (start 73.1 48.913079) (end 73.1 49.535) (width 0.254) (layer "F.Cu") (net 44))
   (segment (start 73.213079 47) (end 73 47) (width 0.254) (layer "F.Cu") (net 44))
-  (segment (start 67.067209 44.511618) (end 68.353827 43.225) (width 0.254) (layer "F.Cu") (net 44))
+  (segment (start 67.01321 44.58679) (end 67.067209 44.532791) (width 0.254) (layer "F.Cu") (net 44))
+  (segment (start 67.067209 44.532791) (end 68.111618 44.532791) (width 0.254) (layer "F.Cu") (net 44))
   (segment (start 74.113079 47.9) (end 73.1 48.913079) (width 0.254) (layer "F.Cu") (net 44))
   (segment (start 77.9 48.966) (end 76.834 47.9) (width 0.254) (layer "F.Cu") (net 44))
   (segment (start 75.975 55.1) (end 76.895666 54.179334) (width 0.254) (layer "F.Cu") (net 44))
   (segment (start 68.85 47) (end 73 47) (width 0.254) (layer "F.Cu") (net 44))
-  (segment (start 67.067209 44.511618) (end 67.067209 44.532791) (width 0.254) (layer "F.Cu") (net 44))
   (segment (start 79.5 86.04) (end 78.436 87.104) (width 0.254) (layer "F.Cu") (net 44))
   (segment (start 66.104 87.104) (end 66 87) (width 0.254) (layer "F.Cu") (net 44))
